File: armpofo_cpu/armpofo_cpu.sch (KiCad schematic (older format))
At the start: 6 parts

Commit message: cpu + ext pins finished
Parts:
- added J?: Conn_02x16_Odd_Even, symbol Connector_Generic:Conn_02x16_Odd_Even
- added J?: Conn_01x08, symbol Connector_Generic:Conn_01x08
Connections:
- net GND: now also U?.10 (VSS), U?.19 (VSSA), U?.26 (VSS), U?.4 (GND), U?.49 (VSS), U?.74 (VSS), U?.99 (VSS), J?.1 (Pin_1), J?.3 (Pin_3), J?.31 (Pin_31), J?.32 (Pin_32), J?.4 (Pin_4)
- net KEY-C1: now also U?.95 (PB8)
- net KEY-C2: now also U?.96 (PB9)
- net KEY-C3: now also U?.97 (PE0)
- net KEY-C4: now also U?.98 (PE1)
- net KEY-C5: now also U?.2 (PE3)
- net KEY-C6: now also U?.3 (PE4)
- net KEY-C7: now also U?.4 (PE5)
- net KEY-C8: now also U?.5 (PE6)
- net KEY-R1: now also U?.77 (PA15)
- net KEY-R2: now also U?.84 (PD3)
- net KEY-R3: now also U?.85 (PD4)
- net KEY-R4: now also U?.86 (PD5)
- net KEY-R5: now also U?.87 (PD6)
- net KEY-R6: now also U?.88 (PD7)
- net KEY-R7: now also U?.89 (PB3)
- net KEY-R8: now also U?.90 (PB4)
- net LCD-CON-PWM: now also U?.34 (PB0)
- net LCD-CS: now also U?.56 (PD9)
- net LCD-D0: now also U?.38 (PE8)
- net LCD-D1: now also U?.39 (PE9)
- net LCD-D2: now also U?.40 (PE10)
- net LCD-D3: now also U?.41 (PE11)
- net LCD-D4: now also U?.42 (PE12)
- net LCD-D5: now also U?.43 (PE13)
- net LCD-D6: now also U?.44 (PE14)
- net LCD-D7: now also U?.45 (PE15)
- net LCD-E: now also U?.35 (PB1)
- net LCD-RS: now also U?.37 (PE7)
- net SOUND-LATCH: now also U?.57 (PD10)
- net QSPI-IO2: now reaches U?.1 (PE2)
- net QSPI-IO2: now also U?.3 (IO2)
- net RESET: now reaches U?.14 (NRST)
- net RESET: now also J?.2 (Pin_2)
- net PC1: now reaches U?.16 (PC1)
- net PC1: now also J?.24 (Pin_24)
- net ADC_VBAT: now reaches U?.18 (PC3_C)
- net PA0: now reaches U?.22 (PA0)
- net PA0: now also J?.7 (Pin_7)
- net PA1: now reaches U?.23 (PA1)
- net PA1: now also J?.9 (Pin_9)
- net PA2: now reaches U?.24 (PA2)
- net PA2: now also J?.11 (Pin_11)
- net PA3: now reaches U?.25 (PA3)
- net PA3: now also J?.13 (Pin_13)
- net PA4: now reaches U?.28 (PA4)
- net PA4: now also J?.15 (Pin_15)
- net PA5: now reaches U?.29 (PA5)
- net PA5: now also J?.17 (Pin_17)
- net PA6: now reaches U?.30 (PA6)
- net PA6: now also J?.19 (Pin_19)
- net PA7: now reaches U?.31 (PA7)
- net PA7: now also J?.21 (Pin_21)
- net PC4: now reaches U?.32 (PC4)
- net PC4: now also J?.26 (Pin_26)
- net PC5: now reaches U?.33 (PC5)
- net PC5: now also J?.28 (Pin_28)
- net QSPI-CLK: now reaches U?.36 (PB2)
- net QSPI-CLK: now also U?.6 (CLK)
- net QSPI-CS: now reaches U?.46 (PB10)
- net QSPI-CS: now also U?.1 (~CS)
- net PB11: now reaches U?.47 (PB11)
- net PB11: now also J?.14 (Pin_14)
- net PB12: now reaches U?.51 (PB12)
- net PB12: now also J?.16 (Pin_16)
- net PB13: now reaches U?.52 (PB13)
- net PB13: now also J?.18 (Pin_18)
- net PB14: now reaches U?.53 (PB14)
- net PB14: now also J?.20 (Pin_20)
- net PB15: now reaches U?.54 (PB15)
- net PB15: now also J?.22 (Pin_22)
- net LCD-R|~w: now reaches U?.55 (PD8)
- net QSPI-IO0: now reaches U?.58 (PD11)
- net QSPI-IO0: now also U?.5 (DI(IO0))
- net QSPI-IO1: now reaches U?.59 (PD12)
- net QSPI-IO1: now also U?.2 (DO(IO1))
- net QSPI-IO3: now reaches U?.60 (PD13)
- net QSPI-IO3: now also U?.7 (IO3)
- net SDCARD-D0: now reaches U?.65 (PC8)
- net SDCARD-D0: now also J?.7 (DAT0)
- net SDCARD-D1: now reaches U?.66 (PC9)
- net SDCARD-D1: now also J?.8 (DAT1)
- net PA8: now reaches U?.67 (PA8)
- net PA8: now also J?.23 (Pin_23)
- net TRACE-TX: now reaches U?.68 (PA9)
- net TRACE-TX: now also J?.8 (Pin_8)
- net TRACE-RX: now reaches U?.69 (PA10)
- net TRACE-RX: now also J?.7 (Pin_7)
- net WAKEUP: now reaches U?.7 (PC13)
- net USB-DM: now reaches U?.70 (PA11)
- net USB-DM: now also J?.2 (D-)
- net USB-DP: now reaches U?.71 (PA12)
- net USB-DP: now also J?.3 (D+)
- net SWDIO: now reaches U?.72 (PA13)
- net SWDIO: now also J?.6 (Pin_6)
- net SWDC: now reaches U?.76 (PA14)
- net SWDC: now also J?.5 (Pin_5)
- net SDCARD-D2: now reaches U?.78 (PC10)
- net SDCARD-D2: now also J?.1 (DAT2)
- net SDCARD-D3: now reaches U?.79 (PC11)
- net SDCARD-D3: now also J?.2 (DAT3/CD)
- net SDCARD-CK: now reaches U?.80 (PC12)
- net SDCARD-CK: now also J?.5 (CLK)
- net PD0: now reaches U?.81 (PD0)
- net PD0: now also J?.25 (Pin_25)
- net PD1: now reaches U?.82 (PD1)
- net PD1: now also J?.27 (Pin_27)
- net SDCARD-CMD: now reaches U?.83 (PD2)
- net SDCARD-CMD: now also J?.3 (CMD)
- net PB5: now reaches U?.91 (PB5)
- net PB5: now also J?.8 (Pin_8)
- net PB6: now reaches U?.92 (PB6)
- net PB6: now also J?.10 (Pin_10)
- net PB7: now reaches U?.93 (PB7)
- net PB7: now also J?.12 (Pin_12)
- net BOOT0: now reaches U?.94 (BOOT0)
- net BOOT0: now also J?.4 (Pin_4)
- net +3V3: now reaches U?.8 (VCC)
- new net 3V3: J?.29 (Pin_29), J?.3 (Pin_3), J?.30 (Pin_30), J?.5 (Pin_5), J?.6 (Pin_6)
- new net 5VINT: J?.1 (Pin_1), J?.2 (Pin_2)
- no-connect marks 0 -> 6
Other:
- note added: "EXTOSC_32k"
- note added: "EXTOSC_HS"
- moved on the sheet: J?

Commit message: schematic almost finished
Parts:
- added C? (x2): 10uF, Capacitor_SMD:C_1210_3225Metric, symbol Device:C_Small
- added C? (x4): 22pF, Capacitor_SMD:C_0603_1608Metric, symbol Device:C
- added C? (x9): 100nF, Capacitor_SMD:C_0603_1608Metric, symbol Device:C
- added C? (x4): 4.7uF, Capacitor_SMD:C_0603_1608Metric, symbol Device:C
- added C? (x2): 100nF, Capacitor_SMD:C_0603_1608Metric, symbol Device:C_Small
- added C? (x2): 22uF/10V, Capacitor_SMD:C_1210_3225Metric, symbol Device:C
- added C?: 470pF, Capacitor_SMD:C_0603_1608Metric, symbol Device:C
- added D?: RED, Diode_SMD:D_0603_1608Metric, symbol Device:LED_ALT
- added D?: SS24, Diode_SMD:D_1206_3216Metric, symbol Device:D_Schottky
- added FB?: 100R, Inductor_SMD:L_0603_1608Metric, symbol Device:Ferrite_Bead_Small
- added J? (x2): Conn_01x01, symbol Connector_Generic:Conn_01x01
- added L?: 2.2 uH, Inductor_SMD:L_1210_3225Metric_Pad1.42x2.65mm_HandSolder, symbol Device:L_Core_Ferrite
- added Q? (x2): Q_PMOS_GDS, symbol Device:Q_PMOS_GDS
- added Q?: Q_NMOS_GDS, symbol Device:Q_NMOS_GDS
- added R? (x11): 100k, Resistor_SMD:R_0603_1608Metric, symbol Device:R
- added R? (x2): 10k, Resistor_SMD:R_0603_1608Metric, symbol Device:R
- added R?: 1k, Resistor_SMD:R_0603_1608Metric, symbol Device:R
- added R?: 22k, Resistor_SMD:R_0603_1608Metric, symbol Device:R
- added U?: TLV62568DBV, Package_TO_SOT_SMD:SOT-23-5, symbol Regulator_Switching:TLV62568DBV
- added Y?: 25MHz, Crystal:Crystal_SMD_3225-4Pin_3.2x2.5mm, symbol Device:Crystal_GND24
- added Y?: 32.768 kHz, symbol Device:Crystal
Connections:
- net 3V3 is gone; now on net +3V3: J?.29 (Pin_29), J?.3 (Pin_3), J?.30 (Pin_30), J?.5 (Pin_5), J?.6 (Pin_6)
- net +3V3: now also J?.4 (VDD), U?.100 (VDD), U?.11 (VDD), U?.21 (VDDA), U?.27 (VDD), U?.50 (VDD), U?.6 (VBAT), U?.75 (VDD), C?.1, C?.1, C?.1, C?.1, C?.1, C?.1, C?.1, C?.1, C?.1, C?.1, C?.1, C?.1, L?.2, R?.1, R?.2, R?.2, R?.2, R?.2, R?.2, R?.2, R?.2, R?.2
- net 5VINT: now also C?.1, C?.1, C?.1, C?.1, D?.1 (K), Q?.2 (D), Q?.3 (S), R?.1, R?.2, U?.1 (EN), U?.4 (VIN)
- net ADC_VBAT: now also R?.1, R?.2
- net BOOT0: now also R?.2
- net GND: now also J?.5 (GND), J?.6 (VSS), C?.2, C?.2, C?.2, C?.2, C?.2, C?.2, C?.2, C?.2, C?.2, C?.2, C?.2, C?.2, C?.2, C?.2, C?.2, C?.2, C?.2, C?.2, C?.2, C?.2, C?.2, C?.2, C?.2, C?.2, J?.1 (Pin_1), Q?.3 (S), R?.1, R?.1, R?.2, R?.2, U?.2 (GND), Y?.2, Y?.4
- net LCD-5V: now also Q?.2 (D)
- net QSPI-CS: now also R?.1
- net RESET: now also C?.1, R?.1
- net SDCARD-CMD: now also R?.1
- net SDCARD-D0: now also R?.1
- net SDCARD-D1: now also R?.1
- net SDCARD-D2: now also R?.1
- net SDCARD-D3: now also R?.1
- net OSC-IN: now reaches U?.12 (PH0)
- net OSC-IN: now also C?.1, Y?.3
- net OSC-OUT: now reaches U?.13 (PH1)
- net OSC-OUT: now also C?.1, Y?.1
- net LED1: now reaches U?.15 (PC0)
- net LED1: now also D?.1 (K)
- net at U?.20 (VREF+): now also C?.1
- net at U?.48 (VCAP1): now also C?.1
- net LCD-ON: now reaches U?.63 (PC6)
- net LCD-ON: now also Q?.1 (G)
- net at U?.73 (VCAP2): now also C?.1
- net at U?.8 (PC14): now also C?.1, Y?.1
- net at U?.9 (PC15): now also C?.1, Y?.2
- net Earth_Protective: now reaches J?.9 (SHIELD)
- net Earth_Protective: now also J?.6 (Shield)
- net USB5V: now reaches J?.1 (VBUS)
- net USB5V: now also FB?.2
- new net: D?.2 (A), FB?.1, Q?.1 (G), R?.2
- new net: D?.2 (A), R?.1
- new net: L?.1, U?.3 (SW)
- new net: R?.1, R?.2, U?.5 (FB)
- new net: Q?.1 (G), Q?.2 (D), R?.1
- new net BAT+: J?.1 (Pin_1), Q?.3 (S)
- no-connect marks 6 -> 5
Other:
- note added: "DEBUG"
- note added: "Extension"
- note removed: "EXTOSC_32k"
- note removed: "EXTOSC_HS"
- moved on the sheet: J?, U?

Commit message: cpu schematic finished
Parts:
- removed C?: 10uF, Capacitor_SMD:C_1210_3225Metric, symbol Device:C_Small
- removed C?: 100nF, Capacitor_SMD:C_0603_1608Metric, symbol Device:C_Small
- removed C?: 4.7uF, Capacitor_SMD:C_0603_1608Metric, symbol Device:C
- removed Q?: Q_NMOS_GDS, symbol Device:Q_NMOS_GDS
- removed U?: STM32H750VBTx, Package_QFP:LQFP-100_14x14mm_P0.5mm, symbol MCU_ST_STM32H7:STM32H750VBTx
- added C11: 470pF, Capacitor_SMD:C_0603_1608Metric, symbol Device:C
- added C12, C13, C19: 22uF/10V, Capacitor_SMD:C_1210_3225Metric, symbol Device:C
- added C18, C24, C27, C8: 100nF, Capacitor_SMD:C_0603_1608Metric, symbol Device:C
- added C25, C9: 4.7uF, Capacitor_SMD:C_0603_1608Metric, symbol Device:C
- added D2: SS24, Diode_SMD:D_1206_3216Metric, symbol Device:D_Schottky
- added FB1: 220R, Inductor_SMD:L_0603_1608Metric, symbol Device:Ferrite_Bead_Small
- added L1: 2.2 uH, Inductor_SMD:L_1210_3225Metric_Pad1.42x2.65mm_HandSolder, symbol Device:L_Core_Ferrite
- added L3: 10 uH, Inductor_SMD:L_1210_3225Metric_Pad1.42x2.65mm_HandSolder, symbol Device:L_Core_Ferrite
- added Q3: Q_PMOS_GDS, Package_TO_SOT_SMD:SOT-23, symbol Device:Q_PMOS_GDS
- added R10: 0.1R, Resistor_SMD:R_0603_1608Metric, symbol Device:R
- added R11, R12: 100k, Resistor_SMD:R_0603_1608Metric, symbol Device:R
- added R16, R18, R4, R8: 0R, Resistor_SMD:R_0603_1608Metric, symbol Device:R
- added R17: 47k, Resistor_SMD:R_0603_1608Metric, symbol Device:R
- added R3: 200k, Resistor_SMD:R_0603_1608Metric, symbol Device:R
- added R7: 22k, Resistor_SMD:R_0603_1608Metric, symbol Device:R
- added U1: TPS63802, Package_SO:TSSOP-10_3x3mm_P0.5mm, symbol PROJECT_LOCAL:TPS63802
- added U3: INA181, Package_TO_SOT_SMD:SOT-23-6, symbol Amplifier_Current:INA181
- added U4: STM32H750VB, Package_QFP:LQFP-100_14x14mm_P0.5mm, symbol PROJECT_LOCAL:STM32H750VB
- J1: renamed from J?; footprint (none) -> Connector_USB:USB_Micro-B_Molex-105017-0001
- J2, J3: renamed from J?; footprint (none) -> Connector_PinHeader_2.54mm:PinHeader_1x01_P2.54mm_Vertical
- J4: renamed from J?; footprint (none) -> Connector_FFC-FPC:TE_1-84953-6_1x16-1MP_P1.0mm_Horizontal
- J5: renamed from J?; footprint (none) -> Connector_FFC-FPC:TE_2-84952-0_1x20-1MP_P1.0mm_Horizontal
- J6: renamed from J?; footprint (none) -> Connector_PinSocket_2.54mm:PinSocket_2x16_P2.54mm_Horizontal
- J7: renamed from J?; footprint (none) -> Connector_PinHeader_2.54mm:PinHeader_1x08_P2.54mm_Horizontal
- J8: renamed from J?; footprint (none) -> PROJECT_LOCAL:Conn_uSDcard
- Q1, Q2: renamed from Q?; footprint (none) -> Package_TO_SOT_SMD:SOT-23
- R15, R9: renamed from R?; value 100k -> 47k
- U5: renamed from U?; footprint Package_SO:SOIC-8_5.23x5.23mm_P1.27mm -> Package_SO:SO-8_5.3x6.2mm_P1.27mm
- Y2: renamed from Y?; footprint (none) -> Crystal:Crystal_DS26_D2.0mm_L6.0mm_Horizontal_1EP_style1
- gave numbers to parts that had none: 40
Connections:
- net +3V3: now also FB1.2, U4.100 (VDD), U4.11 (VDD), U4.27 (VDD), U4.50 (VDD), U4.6 (VBAT), U4.75 (VDD)
- net 5VINT: now also C11.1, C12.1, C13.1, Q3.3 (S), R17.2, R3.1, U1.6 (VOUT); no longer C14.1, D1.1 (K), Q1.2 (D), R13.1
- net BAT+: now also R13.1, R10.1, U3.4 (-); no longer Q1.3 (S)
- net BOOT0: now also U4.94 (BOOT0)
- net GND: now also C11.2, C12.2, C13.2, C18.2, C19.2, C24.2, C25.2, C27.2, C8.2, C9.2, R12.2, R7.2, R8.2, U1.3 (AGND), U1.8 (GND), U3.2 (GND), U4.10 (VSS), U4.19 (VSSA), U4.26 (VSS), U4.49 (VSS), U4.74 (VSS), U4.99 (VSS); no longer R9.1
- net KEY-C1: now also U4.95 (PB8)
- net KEY-C2: now also U4.96 (PB9)
- net KEY-C3: now also U4.97 (PE0)
- net KEY-C4: now also U4.98 (PE1)
- net KEY-C5: now also U4.2 (PE3)
- net KEY-C6: now also U4.3 (PE4)
- net KEY-C7: now also R16.1, U4.4 (PE5)
- net KEY-C8: now also U4.5 (PE6)
- net KEY-R1: now also U4.77 (PA15)
- net KEY-R2: now also U4.84 (PD3)
- net KEY-R3: now also U4.85 (PD4)
- net KEY-R4: now also U4.86 (PD5)
- net KEY-R5: now also U4.87 (PD6)
- net KEY-R6: now also U4.88 (PD7)
- net KEY-R7: now also U4.89 (PB3)
- net KEY-R8: now also U4.90 (PB4)
- net LCD-CON-PWM: now also Q3.1 (G), R17.1, R18.2, U4.34 (PB0); no longer J5.12 (Pin_12)
- net LCD-CS: now also U4.56 (PD9)
- net LCD-D0: now also U4.38 (PE8)
- net LCD-D1: now also U4.39 (PE9)
- net LCD-D2: now also U4.40 (PE10)
- net LCD-D3: now also U4.41 (PE11)
- net LCD-D4: now also U4.42 (PE12)
- net LCD-D5: now also U4.43 (PE13)
- net LCD-D6: now also U4.44 (PE14)
- net LCD-D7: now also U4.45 (PE15)
- net LCD-E: now also U4.35 (PB1)
- net LCD-ON: now also Q2.1 (G), R15.1, U4.63 (PC6)
- net LCD-RS: now also U4.37 (PE7)
- net LED1: now also U4.15 (PC0)
- net OSC-IN: now also U4.12 (PH0)
- net OSC-OUT: now also U4.13 (PH1)
- net PA0: now also U4.22 (PA0)
- net PA1: now also U4.23 (PA1)
- net PA2: now also U4.24 (PA2)
- net PA3: now also U4.25 (PA3)
- net PA4: now also U4.28 (PA4)
- net PA5: now also U4.29 (PA5)
- net PA6: now also U4.30 (PA6)
- net PA7: now also U4.31 (PA7)
- net PA8: now also U4.67 (PA8)
- net PB11: now also U4.47 (PB11)
- net PB12: now also U4.51 (PB12)
- net PB13: now also U4.52 (PB13)
- net PB14: now also U4.53 (PB14)
- net PB15: now also U4.54 (PB15)
- net PB5: now also U4.91 (PB5)
- net PB6: now also U4.92 (PB6)
- net PB7: now also U4.93 (PB7)
- net PC1: now also U4.16 (PC1)
- net PC4: now also U4.32 (PC4)
- net PC5: now also U4.33 (PC5)
- net PD0: now also U4.81 (PD0)
- net PD1: now also U4.82 (PD1)
- net QSPI-CLK: now also U4.36 (PB2)
- net QSPI-CS: now also U4.46 (PB10)
- net QSPI-IO0: now also U4.58 (PD11)
- net QSPI-IO1: now also U4.59 (PD12)
- net QSPI-IO2: now also U4.1 (PE2)
- net QSPI-IO3: now also U4.60 (PD13)
- net RESET: now also U4.14 (NRST)
- net SDCARD-CK: now also U4.80 (PC12)
- net SDCARD-CMD: now also U4.83 (PD2)
- net SDCARD-D0: now also U4.65 (PC8)
- net SDCARD-D1: now also U4.66 (PC9)
- net SDCARD-D2: now also U4.78 (PC10)
- net SDCARD-D3: now also U4.79 (PC11)
- net SOUND-LATCH: now also U4.57 (PD10)
- net SWDC: now also U4.76 (PA14)
- net SWDIO: now also U4.72 (PA13)
- net TRACE-RX: now also U4.69 (PA10)
- net TRACE-TX: now also U4.68 (PA9)
- net USB-DM: now also U4.70 (PA11)
- net USB-DP: now also U4.71 (PA12)
- net USB5V: now also D1.2 (A), FB2.1, Q1.3 (S), R9.2, C18.1, C19.1; no longer FB2.2, J1.1 (VBUS)
- net WAKEUP: now also R16.2, U4.7 (PC13)
- net at C21.1: now also U4.48 (VCAP1)
- net at C22.1: now also U4.73 (VCAP2)
- net at C28.1, Y2.1: now also U4.8 (PC14)
- net at C29.1, Y2.2: now also U4.9 (PC15)
- net ADC_VBAT renamed ADC-BAT
- net ADC-BAT: now also U4.18 (PC3_C)
- net LCD-R\~w renamed LCD-R~W
- net LCD-R~W: now also U4.55 (PD8)
- new net: J5.12 (Pin_12), Q3.2 (D), R18.1
- new net: FB2.2, J1.1 (VBUS)
- new net: L3.1, Q1.2 (D)
- new net: R4.2, R8.1, U1.2 (MODE)
- new net: R3.2, R7.1, U1.4 (FB)
- new net: L1.2, U1.7 (L2)
- new net: L1.1, U1.9 (L1)
- new net: C25.1, D2.2 (A), L3.2, R10.2, U3.3 (+)
- new net: R11.2, R12.1, U3.5 (REF)
- new net 5V-INPUT: C14.1, D1.1 (K), D2.1 (K), R4.1, U1.1 (EN), U1.10 (VIN)
- new net CHARGE-PWM: Q1.1 (G), R9.1, U4.64 (PC7)
- new net I-CHARGE: U3.1, U4.17 (PC2_C)
- new net VDDA: C24.1, C27.1, C8.1, C9.1, FB1.1, R11.1, U3.6 (V+), U4.20 (VREF+), U4.21 (VDDA)
- no-connect marks 5 -> 4
Other:
- note added: "5V tolerant + Open-Drain\nMCU pin required"
- note added: "FPM/PWM\n(more ripple \nat low loads)"
- note added: "PWM Mode"
- note added: "SPACE: R3/C7, ATARI: R7/C7\nFor WAKEUP: R3,R7: output+high, C7: input+pulldown"
- note added: "height\nmax 4 mm"
- moved on the sheet: C1, C10, C14, C15, C16, C17, C2, C20, C21, C22, C23, C26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

Commit message: - CPU board finalisch edge cuts - Keyboard mounting modified to 2.2 mm holes
Parts:
- added H1, H2, H3, H4: 2mm, MountingHole:MountingHole_2.2mm_M2_DIN965_Pad, symbol Mechanical:MountingHole_Pad
- J6: footprint Connector_PinSocket_2.54mm:PinSocket_2x16_P2.54mm_Horizontal -> PROJECT_LOCAL:Conn_Edge_PinSocket_2x16_2.54mm
Connections:
- net Earth_Protective: now also H1.1, H2.1, H3.1, H4.1
Changed lines of the file:
@@
 F 0 "J6" H 14750 9617 50  0000 C CNN
 F 1 "Conn_02x16_Odd_Even" H 14750 9526 50  0000 C CNN
-F 2 "Connector_PinSocket_2.54mm:PinSocket_2x16_P2.54mm_Horizontal" H 14700 8700 50  0001 C CNN
+F 2 "PROJECT_LOCAL:Conn_Edge_PinSocket_2x16_2.54mm" H 14700 8700 50  0001 C CNN
 F 3 "~" H 14700 8700 50  0001 C CNN
 	1    14700 8700
@@
 Wire Wire Line
 	10200 6900 10600 6900
+$Comp
+L Mechanical:MountingHole_Pad H1
+U 1 1 5F9762F5
+P 3500 8900
+F 0 "H1" H 3600 8949 50  0000 L CNN
+F 1 "2mm" H 3600 8858 50  0000 L CNN
+F 2 "MountingHole:MountingHole_2.2mm_M2_DIN965_Pad" H 3500 8900 50  0001 C CNN
+F 3 "~" H 3500 8900 50  0001 C CNN
+	1    3500 8900
+	1    0    0    -1
+$EndComp
+$Comp
+L Mechanical:MountingHole_Pad H2
+U 1 1 5F976D56
+P 4000 8900
+F 0 "H2" H 4100 8949 50  0000 L CNN
+F 1 "2mm" H 4100 8858 50  0000 L CNN
+F 2 "MountingHole:MountingHole_2.2mm_M2_DIN965_Pad" H 4000 8900 50  0001 C CNN
+F 3 "~" H 4000 8900 50  0001 C CNN
+	1    4000 8900
+	1    0    0    -1
+$EndComp
+$Comp
+L Mechanical:MountingHole_Pad H3
+U 1 1 5F976F04
+P 4500 8900
+F 0 "H3" H 4600 8949 50  0000 L CNN
+F 1 "2mm" H 4600 8858 50  0000 L CNN
+F 2 "MountingHole:MountingHole_2.2mm_M2_DIN965_Pad" H 4500 8900 50  0001 C CNN
+F 3 "~" H 4500 8900 50  0001 C CNN
+	1    4500 8900
+	1    0    0    -1
+$EndComp
+$Comp
+L power:Earth_Protective #PWR?
+U 1 1 5F9BEB64
+P 4000 9100
+AR Path="/5FD2A278/5F9BEB64" Ref="#PWR?"  Part="1"
+AR Path="/5F9BEB64" Ref="#PWR0101"  Part="1"
+F 0 "#PWR0101" H 4250 8850 50  0001 C CNN
+F 1 "Earth_Protective" H 4450 8950 50  0001 C CNN
+F 2 "" H 4000 9000 50  0001 C CNN
+F 3 "~" H 4000 9000 50  0001 C CNN
+	1    4000 9100
+	-1   0    0    -1
+$EndComp
+Wire Wire Line
+	3500 9000 4000 9000
+Connection ~ 4000 9000
+Wire Wire Line
+	4000 9000 4500 9000
+Wire Wire Line
+	4000 9000 4000 9100
+$Comp
+L Mechanical:MountingHole_Pad H4
+U 1 1 5F9D6D76
+P 5000 8900
+F 0 "H4" H 5100 8949 50  0000 L CNN
+F 1 "2mm" H 5100 8858 50  0000 L CNN
+F 2 "MountingHole:MountingHole_2.2mm_M2_DIN965_Pad" H 5000 8900 50  0001 C CNN
+F 3 "~" H 5000 8900 50  0001 C CNN
+	1    5000 8900
+	1    0    0    -1
+$EndComp
+Wire Wire Line
+	4500 9000 5000 9000
+Connection ~ 4500 9000
 $EndSCHEMATC

Commit message: some progress
Parts:
- added C32: 1nF, Capacitor_SMD:C_0603_1608Metric, symbol Device:C
- added D4: SS24, Diode_SMD:D_1206_3216Metric, symbol Device:D_Schottky
- added J9: Conn_01x01, Connector_PinHeader_2.54mm:PinHeader_1x01_P2.54mm_Vertical, symbol Connector_Generic:Conn_01x01
- added R19, R27: 100k, Resistor_SMD:R_0603_1608Metric, symbol Device:R
- added R28, R29: 22R, Resistor_SMD:R_0603_1608Metric, symbol Device:R
- U1: footprint Package_SO:TSSOP-10_3x3mm_P0.5mm -> PROJECT_LOCAL:DLA0010A
Connections:
- net BAT+: now also C32.2
- net GND: now also D4.2 (A), J9.1 (Pin_1), R27.2
- net LED1: now also U4.62 (PD15); no longer U4.15 (PC0)
- net USB-DM: now also R29.2; no longer J1.2 (D-)
- net USB-DP: now also R28.2; no longer J1.3 (D+)
- net USB5V: now also R19.1
- net at L3.1, Q1.2 (D): now also D4.1 (K)
- net at C25.1, D2.2 (A), L3.2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: now also C32.1
- net 5V-INPUT renamed 3-5V
- new net: J1.2 (D-), R29.1
- new net: J1.3 (D+), R28.1
- new net ADC-5V: R19.2, R27.1, U4.15 (PC0)
- no-connect marks 4 -> 3
Other:
- moved on the sheet: C11, C12, C13, C14, C15, C16, C17, C18, C19, C20, C24, C25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

Commit message: routing progress 70%
Parts:
- removed C27: 100nF, Capacitor_SMD:C_0603_1608Metric, symbol Device:C
- removed R8: 0R, Resistor_SMD:R_0603_1608Metric, symbol Device:R
- removed U1: TPS63802, PROJECT_LOCAL:DLA0010A, symbol PROJECT_LOCAL:TPS63802
- added C33: 100nF, Capacitor_SMD:C_0603_1608Metric, symbol Device:C_Small
- added J10: Conn_01x16, Connector_PinHeader_1.27mm:PinHeader_1x16_P1.27mm_Vertical, symbol Connector_Generic:Conn_01x16
- added J11: Conn_01x20, Connector_PinHeader_1.27mm:PinHeader_1x20_P1.27mm_Vertical, symbol Connector_Generic:Conn_01x20
- added U1: TPS63030DSK, Package_SON:WSON-10-1EP_2.5x2.5mm_P0.5mm_EP1.2x2mm, symbol Regulator_Switching:TPS63030DSK
- R10: footprint Resistor_SMD:R_0603_1608Metric -> Resistor_SMD:R_1206_3216Metric
- R4: value 0R -> 1k
Connections:
- net +3V3: now also D3.2 (A); no longer R25.2
- net 3-5V: now also U1.5 (VIN); no longer R4.1
- net 5VINT: now also U1.1 (VOUT)
- net BAT+: no longer C32.2
- net Earth_Protective: no longer H1.1, H2.1, H3.1, H4.1
- net GND: now also C32.2, C33.2, J11.18 (Pin_18), J11.19 (Pin_19), J11.20 (Pin_20), U1.11 (PGND), U1.3 (PGND), U1.9 (GND)
- net I-CHARGE: now also C32.1, R4.2; no longer U3.1
- net KEY-C1: now also J10.9 (Pin_9)
- net KEY-C2: now also J10.10 (Pin_10)
- net KEY-C3: now also J10.11 (Pin_11)
- net KEY-C4: now also J10.12 (Pin_12)
- net KEY-C5: now also J10.13 (Pin_13)
- net KEY-C6: now also J10.14 (Pin_14)
- net KEY-C7: now also J10.15 (Pin_15)
- net KEY-C8: now also J10.16 (Pin_16)
- net KEY-R1: now also J10.1 (Pin_1)
- net KEY-R2: now also J10.2 (Pin_2)
- net KEY-R3: now also J10.3 (Pin_3)
- net KEY-R4: now also J10.4 (Pin_4)
- net KEY-R5: now also J10.5 (Pin_5)
- net KEY-R6: now also J10.6 (Pin_6)
- net KEY-R7: now also J10.7 (Pin_7)
- net KEY-R8: now also J10.8 (Pin_8)
- net LCD-5V: now also J11.1 (Pin_1), J11.2 (Pin_2), J11.3 (Pin_3)
- net LCD-CS: now also J11.16 (Pin_16)
- net LCD-D0: now also J11.4 (Pin_4)
- net LCD-D1: now also J11.5 (Pin_5)
- net LCD-D2: now also J11.6 (Pin_6)
- net LCD-D3: now also J11.7 (Pin_7)
- net LCD-D4: now also J11.8 (Pin_8)
- net LCD-D5: now also J11.9 (Pin_9)
- net LCD-D6: now also J11.10 (Pin_10)
- net LCD-D7: now also J11.11 (Pin_11)
- net LCD-E: now also J11.15 (Pin_15)
- net LCD-RS: now also J11.14 (Pin_14)
- net LCD-R~W: now also J11.17 (Pin_17)
- net LED1: now also R25.1; no longer D3.1 (K)
- net SOUND-LATCH: now also J11.13 (Pin_13)
- net LCD-CTRPWM: now reaches J5.12 (Pin_12), Q3.2 (D), R18.1
- net LCD-CTRPWM: now also J11.12 (Pin_12)
- net at R3.2, R7.1: now also U1.10 (FB)
- net at L1.2: now also U1.2 (L2)
- net at L1.1: now also U1.4 (L1)
- net at C25.1, D2.2 (A), L3.2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: no longer C32.1
- new net: C33.1, U1.6 (EN), U1.7 (PS/SYNC), U1.8 (VINA)
- new net: R4.1, U3.1
- new net: D3.1 (K), R25.2
- no-connect marks 3 -> 6
Other:
- note removed: "FPM/PWM\n(more ripple \nat low loads)"
- note removed: "PWM Mode"
- moved on the sheet: C30, C31, C32, D3, J4, J5, J8, Q2, Q3, R15, R16, R17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
