File: armpofo_cpu/armpofo_cpu.sch (KiCad schematic (older format))
At the start: 94 parts, among them J1 USB_OTG, J10 Conn_01x16, J11 Conn_01x20, J2 Conn_01x01, J3 Conn_01x01, J4 Conn_01x16, J5 Conn_01x20, J6 Conn_02x16_Odd_Even, J7 Conn_01x08, J8 Micro_SD_Card, J9 Conn_01x01, Q1 Q_PMOS_GDS, Q2 Q_PMOS_GDS, Q3 Q_PMOS_GDS, U1 TPS63030DSK, U2 TLV62568DBV, U3 INA181, U4 STM32H750VB, U5 W25Q32JVSS, Y1 25MHz, Y2 32.768 kHz

Commit message: routing finished.
Connections:
- net PA0: now also J6.8 (Pin_8); no longer J6.7 (Pin_7)
- net PA1: now also J6.7 (Pin_7); no longer J6.9 (Pin_9)
- net PA2: now also J6.10 (Pin_10); no longer J6.11 (Pin_11)
- net PA3: now also J6.9 (Pin_9); no longer J6.13 (Pin_13)
- net PA4: now also J6.12 (Pin_12); no longer J6.15 (Pin_15)
- net PA5: now also J6.11 (Pin_11); no longer J6.17 (Pin_17)
- net PA6: now also J6.14 (Pin_14); no longer J6.19 (Pin_19)
- net PA7: now also J6.13 (Pin_13); no longer J6.21 (Pin_21)
- net PA8: now also J6.16 (Pin_16); no longer J6.23 (Pin_23)
- net PB11: now also J6.20 (Pin_20); no longer J6.14 (Pin_14)
- net PB12: now also J6.19 (Pin_19); no longer J6.16 (Pin_16)
- net PB13: now also J6.22 (Pin_22); no longer J6.18 (Pin_18)
- net PB14: now also J6.21 (Pin_21); no longer J6.20 (Pin_20)
- net PB15: now also J6.24 (Pin_24); no longer J6.22 (Pin_22)
- net PB5: now also J6.15 (Pin_15); no longer J6.8 (Pin_8)
- net PB6: now also J6.18 (Pin_18); no longer J6.10 (Pin_10)
- net PB7: now also J6.17 (Pin_17); no longer J6.12 (Pin_12)
- net PC1: now also J6.23 (Pin_23); no longer J6.24 (Pin_24)
- net PC5: now also J6.25 (Pin_25); no longer J6.28 (Pin_28)
- net PD0: now also J6.28 (Pin_28); no longer J6.25 (Pin_25)
Changed lines of the file:
@@
 L Connector_Generic:Conn_02x16_Odd_Even J6
 U 1 1 5F8D19FF
-P 14700 8700
-F 0 "J6" H 14750 9617 50  0000 C CNN
-F 1 "Conn_02x16_Odd_Even" H 14750 9526 50  0000 C CNN
-F 2 "PROJECT_LOCAL:Conn_Edge_PinSocket_2x16_2.54mm" H 14700 8700 50  0001 C CNN
-F 3 "~" H 14700 8700 50  0001 C CNN
-	1    14700 8700
-	1    0    0    -1
+P 14800 8700
+F 0 "J6" H 14850 9617 50  0000 C CNN
+F 1 "Conn_02x16_Odd_Even" H 14850 9526 50  0000 C CNN
+F 2 "PROJECT_LOCAL:Conn_Edge_PinSocket_2x16_2.54mm" H 14800 8700 50  0001 C CNN
+F 3 "~" H 14800 8700 50  0001 C CNN
+	1    14800 8700
+	-1   0    0    -1
 $EndComp
 Text Label 15500 9100 2    50   ~ 0
 PC1
+Text Label 15500 8300 2    50   ~ 0
+PA1
 Text Label 14000 8400 0    50   ~ 0
-PA1
+PA2
 Text Label 14000 8500 0    50   ~ 0
-PA2
+PA4
+Text Label 15500 8500 2    50   ~ 0
+PA5
+Text Label 15500 8600 2    50   ~ 0
+PA7
+Text Label 14000 9200 0    50   ~ 0
+PC4
+Text Label 15500 9200 2    50   ~ 0
+PC5
+Text Label 14000 8900 0    50   ~ 0
+PB11
+Text Label 15500 8900 2    50   ~ 0
+PB12
+Text Label 14000 9000 0    50   ~ 0
+PB13
+Text Label 15500 9000 2    50   ~ 0
+PB14
+Text Label 14000 9100 0    50   ~ 0
+PB15
 Text Label 14000 8700 0    50   ~ 0
-PA4
+PA8
+Text Label 14000 9300 0    50   ~ 0
+PD0
+Text Label 15500 9300 2    50   ~ 0
+PD1
+Text Label 15500 8700 2    50   ~ 0
+PB5
 Text Label 14000 8800 0    50   ~ 0
-PA5
-Text Label 14000 9000 0    50   ~ 0
-PA7
-Text Label 15500 9200 2    50   ~ 0
-PC4
-Text Label 15500 9300 2    50   ~ 0
-PC5
-Text Label 15500 8600 2    50   ~ 0
-PB11
-Text Label 15500 8700 2    50   ~ 0
-PB12
+PB6
 Text Label 15500 8800 2    50   ~ 0
-PB13
-Text Label 15500 8900 2    50   ~ 0
-PB14
-Text Label 15500 9000 2    50   ~ 0
-PB15
-Text Label 14000 9100 0    50   ~ 0
-PA8
-Text Label 14000 9200 0    50   ~ 0
-PD0
-Text Label 14000 9300 0    50   ~ 0
-PD1
-Text Label 15500 8300 2    50   ~ 0
-PB5
-Text Label 15500 8400 2    50   ~ 0
-PB6
-Text Label 15500 8500 2    50   ~ 0
 PB7
+Text Label 15500 9500 2    50   ~ 0
+GND
+Text Label 15500 8200 2    50   ~ 0
+3V3
+Text Label 15500 8000 2    50   ~ 0
+5VINT
 Text Label 14000 9500 0    50   ~ 0
+GND
+Text Label 14000 8000 0    50   ~ 0
+5VINT
+Text Label 15500 8100 2    50   ~ 0
+GND
+Text Label 14000 8100 0    50   ~ 0
 GND
 Text Label 14000 8200 0    50   ~ 0
 3V3
-Text Label 14000 8000 0    50   ~ 0
-5VINT
-Text Label 15500 9500 2    50   ~ 0
-GND
-Text Label 15500 8000 2    50   ~ 0
-5VINT
-Text Label 14000 8100 0    50   ~ 0
-GND
-Text Label 15500 8100 2    50   ~ 0
-GND
-Text Label 15500 8200 2    50   ~ 0
+Text Label 15500 9400 2    50   ~ 0
 3V3
 Text Label 14000 9400 0    50   ~ 0
 3V3
-Text Label 15500 9400 2    50   ~ 0
-3V3
-Text Label 14000 8900 0    50   ~ 0
+Text Label 14000 8600 0    50   ~ 0
 PA6
 Text Label 14000 8300 0    50   ~ 0
 PA0
-Text Label 14000 8600 0    50   ~ 0
+Text Label 15500 8400 2    50   ~ 0
 PA3
 Wire Wire Line
-	14000 8000 14500 8000
-Wire Wire Line
-	15000 8000 15500 8000
-Wire Wire Line
-	14000 8100 14500 8100
-Wire Wire Line
-	15000 8100 15500 8100
-Wire Wire Line
-	14000 8200 14500 8200
+	15500 8000 15000 8000
+Wire Wire Line
+	14500 8000 14000 8000
+Wire Wire Line
+	15500 8100 15000 8100
+Wire Wire Line
+	14500 8100 14000 8100
+Wire Wire Line
+	15500 8200 15000 8200
+Wire Wire Line
+	15500 8300 15000 8300
+Wire Wire Line
+	15500 8400 15000 8400
+Wire Wire Line
+	15500 8500 15000 8500
+Wire Wire Line
+	15500 8600 15000 8600
+Wire Wire Line
+	15500 8700 15000 8700
+Wire Wire Line
+	15500 8800 15000 8800
+Wire Wire Line
+	15500 8900 15000 8900
+Wire Wire Line
+	15500 9000 15000 9000
+Wire Wire Line
+	15500 9100 15000 9100
+Wire Wire Line
+	15500 9200 15000 9200
+Wire Wire Line
+	15500 9300 15000 9300
+Wire Wire Line
+	15500 9400 15000 9400
+Wire Wire Line
+	15500 9500 15000 9500
+Wire Wire Line
+	14500 8400 14000 8400
+Wire Wire Line
+	14500 8500 14000 8500
+Wire Wire Line
+	14500 8600 14000 8600
+Wire Wire Line
+	14500 8700 14000 8700
+Wire Wire Line
+	14500 8800 14000 8800
+Wire Wire Line
+	14500 8900 14000 8900
+Wire Wire Line
+	14500 9000 14000 9000
+Wire Wire Line
+	14500 9100 14000 9100
+Wire Wire Line
+	14500 9200 14000 9200
+Wire Wire Line
+	14500 9300 14000 9300
+Wire Wire Line
+	14500 9400 14000 9400
+Wire Wire Line
+	14500 9500 14000 9500
+Wire Wire Line
+	14500 8200 14000 8200
 Wire Wire Line
 	14000 8300 14500 8300
-Wire Wire Line
-	14000 8400 14500 8400
-Wire Wire Line
-	14000 8500 14500 8500
-Wire Wire Line
-	14000 8600 14500 8600
-Wire Wire Line
-	14000 8700 14500 8700
-Wire Wire Line
-	14000 8800 14500 8800
-Wire Wire Line
-	14000 8900 14500 8900
-Wire Wire Line
-	14000 9000 14500 9000
-Wire Wire Line
-	14000 9100 14500 9100
-Wire Wire Line
-	14000 9200 14500 9200
-Wire Wire Line
-	14000 9300 14500 9300
-Wire Wire Line
-	14000 9400 14500 9400
-Wire Wire Line
-	14000 9500 14500 9500
-Wire Wire Line
-	15000 8400 15500 8400
-Wire Wire Line
-	15000 8500 15500 8500
-Wire Wire Line
-	15000 8600 15500 8600
-Wire Wire Line
-	15000 8700 15500 8700
-Wire Wire Line
-	15000 8800 15500 8800
-Wire Wire Line
-	15000 8900 15500 8900
-Wire Wire Line
-	15000 9000 15500 9000
-Wire Wire Line
-	15000 9100 15500 9100
-Wire Wire Line
-	15000 9200 15500 9200
-Wire Wire Line
-	15000 9300 15500 9300
-Wire Wire Line
-	15000 9400 15500 9400
-Wire Wire Line
-	15000 9500 15500 9500
-Wire Wire Line
-	15000 8200 15500 8200
-Wire Wire Line
-	15500 8300 15000 8300
 Text Label 5500 1900 2    50   ~ 0
 PA1
@@
 	1    0    0    -1
 $EndComp
-Text Notes 14050 7750 0    50   ~ 0
+Text Notes 15450 7750 2    50   ~ 0
 Extension
 Text Notes 12000 8600 0    50   ~ 0

Commit message: PCB corrections some items moved to the backside
Parts:
- removed J11: Conn_01x20, Connector_PinHeader_1.27mm:PinHeader_1x20_P1.27mm_Vertical, symbol Connector_Generic:Conn_01x20
- L1, L2, L3: footprint Inductor_SMD:L_1210_3225Metric_Pad1.42x2.65mm_HandSolder -> Inductor_SMD:L_Taiyo-Yuden_NR-40xx_HandSoldering
Connections:
- net KEY-C1: now also J4.8 (Pin_8), U4.90 (PB4); no longer J4.9 (Pin_9), U4.95 (PB8)
- net KEY-C2: now also J4.7 (Pin_7), U4.89 (PB3); no longer J4.10 (Pin_10), U4.96 (PB9)
- net KEY-C3: now also J4.6 (Pin_6), U4.88 (PD7); no longer J4.11 (Pin_11), U4.97 (PE0)
- net KEY-C4: now also J4.5 (Pin_5), U4.87 (PD6); no longer J4.12 (Pin_12), U4.98 (PE1)
- net KEY-C5: now also J4.4 (Pin_4), U4.86 (PD5); no longer J4.13 (Pin_13), U4.2 (PE3)
- net KEY-C6: now also J4.3 (Pin_3), U4.85 (PD4); no longer J4.14 (Pin_14), U4.3 (PE4)
- net KEY-C7: now also J4.2 (Pin_2), U4.84 (PD3); no longer J4.15 (Pin_15), U4.4 (PE5)
- net KEY-C8: now also J4.1 (Pin_1), U4.77 (PA15); no longer J4.16 (Pin_16), U4.5 (PE6)
- net KEY-R1: now also J4.16 (Pin_16), U4.5 (PE6); no longer J4.1 (Pin_1), U4.77 (PA15)
- net KEY-R2: now also J4.15 (Pin_15), U4.4 (PE5); no longer J4.2 (Pin_2), U4.84 (PD3)
- net KEY-R3: now also J4.14 (Pin_14), U4.3 (PE4); no longer J4.3 (Pin_3), U4.85 (PD4)
- net KEY-R4: now also J4.13 (Pin_13), U4.2 (PE3); no longer J4.4 (Pin_4), U4.86 (PD5)
- net KEY-R5: now also J4.12 (Pin_12), U4.98 (PE1); no longer J4.5 (Pin_5), U4.87 (PD6)
- net KEY-R6: now also J4.11 (Pin_11), U4.97 (PE0); no longer J4.6 (Pin_6), U4.88 (PD7)
- net KEY-R7: now also J4.10 (Pin_10), U4.96 (PB9); no longer J4.7 (Pin_7), U4.89 (PB3)
- net KEY-R8: now also J4.9 (Pin_9), U4.95 (PB8); no longer J4.8 (Pin_8), U4.90 (PB4)
