File: armpofo_cpu/armpofo_cpu.kicad_pcb (KiCad board)
At the start: 2 copper layers, 184.1 x 74 mm, 94 parts, among them J1 USB_OTG, J10 Conn_01x16, J11 Conn_01x20, J2 Conn_01x01, J3 Conn_01x01, J4 Conn_01x16, J5 Conn_01x20, J6 Conn_02x16_Odd_Even, J7 Conn_01x08, J8 Micro_SD_Card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

Commit message: gerber files generated
Other:
- board text added: "3.3V"
- board text added: "ARMPOFO CPU"
- board text added: "BOOT0"
- board text added: "C1"
- board text added: "R8"
- board text added: "RESET"
- board text added: "STM32H750"
- board text added: "SWDCLK"
- board text added: "SWDIO"
- board text added: "TRACE-RX"
- board text added: "TRACE-TX"
